Commit message: change

File: two_robot/urdf/two_robot.urdf (robot description, URDF)
Before this commit: robot two_robot, 7 links, 6 joints
Links:
- added link camera_link; visual mesh filename=model://kinect/meshes/kinect.dae
Joints:
- added joint camera_joint: type fixed, parent base_link, child camera_link, origin xyz=-0.012 -0.116 0.155 rpy=0 0.62832 3.1416
